Commit message: fix: update yaml load function

File: pixkit_sensor_kit_drscription/urdf/sensors.xacro (robot description, xacro)
@@ -15,5 +15,5 @@
   <link name="ultrasonic_7" />
   <xacro:arg name="config_dir" default="$(find pixkit_sensor_kit_description)"/>
-  <xacro:property name="calibration" value="${load_yaml('$(arg config_dir)/sensors_calibration.yaml')}"/>
+  <xacro:property name="calibration" value="${xacro.load_yaml('$(arg config_dir)/sensors_calibration.yaml')}"/>
  <!-- embedded sensors -->
   <joint name="zed_baselink" type="fixed">

Commit message: feat: add launch file for gnss,imu,lidar. update sensor description

File: pixkit_sensor_kit_drscription/urdf/sensors.xacro (robot description, xacro)
@@ -6,4 +6,5 @@
   <link name="rs16" />
   <link name="rsbp" />
+  <link name="os_sensor" />
   <link name="ultrasonic_0" />
   <link name="ultrasonic_1" />
@@ -17,4 +18,9 @@
   <xacro:property name="calibration" value="${xacro.load_yaml('$(arg config_dir)/sensors_calibration.yaml')}"/>
  <!-- embedded sensors -->
+  <joint name="baselink_os_sensor" type="fixed">
+    <parent link="base_link" />
+    <child link="os_sensor" />
+    <origin xyz="${calibration['base_link2os_sensor']['x']} ${calibration['base_link2os_sensor']['y']} ${calibration['base_link2os_sensor']['z']}" rpy="${calibration['base_link2os_sensor']['roll']} ${calibration['base_link2os_sensor']['pitch']} ${calibration['base_link2os_sensor']['yaw']}" />
+  </joint>
   <joint name="zed_baselink" type="fixed">
     <parent link="base_link" />
