Commit message: feat: use ros2 farm ouster driver, use IMU inside rtk-ins localizer

File: pixkit_sensor_kit_description/urdf/sensors.xacro (robot description, xacro)
@@ -6,4 +6,5 @@
   <link name="rs16" />
   <link name="rsbp" />
+  <link name="gnss" />
   <link name="os_sensor" />
   <link name="ultrasonic_0" />
@@ -37,4 +38,9 @@
     <child link="rs16" />
     <origin xyz="${calibration['base_link2rs16']['x']} ${calibration['base_link2rs16']['y']} ${calibration['base_link2rs16']['z']}" rpy="${calibration['base_link2rs16']['roll']} ${calibration['base_link2rs16']['pitch']} ${calibration['base_link2rs16']['yaw']}" />
+  </joint>
+  <joint name="baselink_gnss" type="fixed">
+    <parent link="base_link" />
+    <child link="gnss" />
+    <origin xyz="${calibration['base_link2gnss']['x']} ${calibration['base_link2gnss']['y']} ${calibration['base_link2gnss']['z']}" rpy="${calibration['base_link2gnss']['roll']} ${calibration['base_link2gnss']['pitch']} ${calibration['base_link2gnss']['yaw']}" />
   </joint>
   <joint name="baselink_ultrasonic_0" type="fixed">

Commit message: feat: add camera launcher to sensing.launch

File: pixkit_sensor_kit_description/urdf/sensors.xacro (robot description, xacro)
@@ -16,4 +16,5 @@
   <link name="ultrasonic_6" />
   <link name="ultrasonic_7" />
+  <link name="camera" />
   <xacro:arg name="config_dir" default="$(find pixkit_sensor_kit_description)"/>
   <xacro:property name="calibration" value="${xacro.load_yaml('$(arg config_dir)/sensors_calibration.yaml')}"/>
@@ -84,3 +85,8 @@
     <origin xyz="${calibration['base_link2ultrasonic_7']['x']} ${calibration['base_link2ultrasonic_7']['y']} ${calibration['base_link2ultrasonic_7']['z']}" rpy="${calibration['base_link2ultrasonic_7']['roll']} ${calibration['base_link2ultrasonic_7']['pitch']} ${calibration['base_link2ultrasonic_7']['yaw']}" />
   </joint>
+  <joint name="rs16_camera" type="fixed">
+    <parent link="rs16" />
+    <child link="camera" />
+    <origin xyz="${calibration['rs162camera']['x']} ${calibration['rs162camera']['y']} ${calibration['rs162camera']['z']}" rpy="${calibration['rs162camera']['roll']} ${calibration['rs162camera']['pitch']} ${calibration['rs162camera']['yaw']}" />
+  </joint>
 </robot>

Commit message: feat: 按照awsim_sensor_kit_launch风格来编写

File: pixkit_sensor_kit_description/urdf/sensors.xacro (robot description, xacro)
@@ -1,92 +1,98 @@
 <?xml version="1.0"?>
-<robot name="vehicle"
-  xmlns:xacro="http://ros.org/wiki/xacro">
-  <link name="zed_base_link" />
-  <!-- <link name="base_link" />  -->
-  <link name="rs16" />
-  <link name="rsbp" />
-  <link name="gnss" />
-  <link name="os_sensor" />
-  <link name="ultrasonic_0" />
-  <link name="ultrasonic_1" />
-  <link name="ultrasonic_2" />
-  <link name="ultrasonic_3" />
-  <link name="ultrasonic_4" />
-  <link name="ultrasonic_5" />
-  <link name="ultrasonic_6" />
-  <link name="ultrasonic_7" />
-  <link name="camera" />
-  <xacro:arg name="config_dir" default="$(find pixkit_sensor_kit_description)"/>
+<robot name="vehicle" xmlns:xacro="http://ros.org/wiki/xacro">
+  <xacro:arg name="config_dir" default="$(find pixkit_sensor_kit_description)/config"/>
   <xacro:property name="calibration" value="${xacro.load_yaml('$(arg config_dir)/sensors_calibration.yaml')}"/>
- <!-- embedded sensors -->
-  <joint name="baselink_os_sensor" type="fixed">
-    <parent link="base_link" />
-    <child link="os_sensor" />
-    <origin xyz="${calibration['base_link2os_sensor']['x']} ${calibration['base_link2os_sensor']['y']} ${calibration['base_link2os_sensor']['z']}" rpy="${calibration['base_link2os_sensor']['roll']} ${calibration['base_link2os_sensor']['pitch']} ${calibration['base_link2os_sensor']['yaw']}" />
-  </joint>
-  <joint name="zed_baselink" type="fixed">
-    <parent link="base_link" />
-    <child link="zed_base_link" />
-    <origin xyz="${calibration['base_link2zed']['x']} ${calibration['base_link2zed']['y']} ${calibration['base_link2zed']['z']}" rpy="${calibration['base_link2zed']['roll']} ${calibration['base_link2zed']['pitch']} ${calibration['base_link2zed']['yaw']}" />
-    </joint>
-  <joint name="baselink_rsbp" type="fixed">
-    <parent link="base_link" />
-    <child link="rsbp" />
-    <origin xyz="${calibration['base_link2rsbp']['x']} ${calibration['base_link2rsbp']['y']} ${calibration['base_link2rsbp']['z']}" rpy="${calibration['base_link2rsbp']['roll']} ${calibration['base_link2rsbp']['pitch']} ${calibration['base_link2rsbp']['yaw']}" />
-  </joint>
-  <joint name="baselink_rs16" type="fixed">
-    <parent link="base_link" />
-    <child link="rs16" />
-    <origin xyz="${calibration['base_link2rs16']['x']} ${calibration['base_link2rs16']['y']} ${calibration['base_link2rs16']['z']}" rpy="${calibration['base_link2rs16']['roll']} ${calibration['base_link2rs16']['pitch']} ${calibration['base_link2rs16']['yaw']}" />
-  </joint>
-  <joint name="baselink_gnss" type="fixed">
-    <parent link="base_link" />
-    <child link="gnss" />
-    <origin xyz="${calibration['base_link2gnss']['x']} ${calibration['base_link2gnss']['y']} ${calibration['base_link2gnss']['z']}" rpy="${calibration['base_link2gnss']['roll']} ${calibration['base_link2gnss']['pitch']} ${calibration['base_link2gnss']['yaw']}" />
-  </joint>
-  <joint name="baselink_ultrasonic_0" type="fixed">
-    <parent link="base_link" />
-    <child link="ultrasonic_0" />
-    <origin xyz="${calibration['base_link2ultrasonic_0']['x']} ${calibration['base_link2ultrasonic_0']['y']} ${calibration['base_link2ultrasonic_0']['z']}" rpy="${calibration['base_link2ultrasonic_0']['roll']} ${calibration['base_link2ultrasonic_0']['pitch']} ${calibration['base_link2ultrasonic_0']['yaw']}" />
-  </joint>
-  <joint name="baselink_ultrasonic_1" type="fixed">
-    <parent link="base_link" />
-    <child link="ultrasonic_1" />
-    <origin xyz="${calibration['base_link2ultrasonic_1']['x']} ${calibration['base_link2ultrasonic_1']['y']} ${calibration['base_link2ultrasonic_1']['z']}" rpy="${calibration['base_link2ultrasonic_1']['roll']} ${calibration['base_link2ultrasonic_1']['pitch']} ${calibration['base_link2ultrasonic_1']['yaw']}" />
-  </joint>
-  <joint name="baselink_ultrasonic_2" type="fixed">
-    <parent link="base_link" />
-    <child link="ultrasonic_2" />
-    <origin xyz="${calibration['base_link2ultrasonic_2']['x']} ${calibration['base_link2ultrasonic_2']['y']} ${calibration['base_link2ultrasonic_2']['z']}" rpy="${calibration['base_link2ultrasonic_2']['roll']} ${calibration['base_link2ultrasonic_2']['pitch']} ${calibration['base_link2ultrasonic_2']['yaw']}" />
-  </joint>
-  <joint name="baselink_ultrasonic_3" type="fixed">
-    <parent link="base_link" />
-    <child link="ultrasonic_3" />
-    <origin xyz="${calibration['base_link2ultrasonic_3']['x']} ${calibration['base_link2ultrasonic_3']['y']} ${calibration['base_link2ultrasonic_3']['z']}" rpy="${calibration['base_link2ultrasonic_3']['roll']} ${calibration['base_link2ultrasonic_3']['pitch']} ${calibration['base_link2ultrasonic_3']['yaw']}" />
-  </joint>
-  <joint name="baselink_ultrasonic_4" type="fixed">
-    <parent link="base_link" />
-    <child link="ultrasonic_4" />
-    <origin xyz="${calibration['base_link2ultrasonic_4']['x']} ${calibration['base_link2ultrasonic_4']['y']} ${calibration['base_link2ultrasonic_4']['z']}" rpy="${calibration['base_link2ultrasonic_4']['roll']} ${calibration['base_link2ultrasonic_4']['pitch']} ${calibration['base_link2ultrasonic_4']['yaw']}" />
-  </joint>
-  <joint name="baselink_ultrasonic_5" type="fixed">
-    <parent link="base_link" />
-    <child link="ultrasonic_5" />
-    <origin xyz="${calibration['base_link2ultrasonic_5']['x']} ${calibration['base_link2ultrasonic_5']['y']} ${calibration['base_link2ultrasonic_5']['z']}" rpy="${calibration['base_link2ultrasonic_5']['roll']} ${calibration['base_link2ultrasonic_5']['pitch']} ${calibration['base_link2ultrasonic_5']['yaw']}" />
-  </joint>
-  <joint name="baselink_ultrasonic_6" type="fixed">
-    <parent link="base_link" />
-    <child link="ultrasonic_6" />
-    <origin xyz="${calibration['base_link2ultrasonic_6']['x']} ${calibration['base_link2ultrasonic_6']['y']} ${calibration['base_link2ultrasonic_6']['z']}" rpy="${calibration['base_link2ultrasonic_6']['roll']} ${calibration['base_link2ultrasonic_6']['pitch']} ${calibration['base_link2ultrasonic_6']['yaw']}" />
-  </joint>
-  <joint name="baselink_ultrasonic_7" type="fixed">
-    <parent link="base_link" />
-    <child link="ultrasonic_7" />
-    <origin xyz="${calibration['base_link2ultrasonic_7']['x']} ${calibration['base_link2ultrasonic_7']['y']} ${calibration['base_link2ultrasonic_7']['z']}" rpy="${calibration['base_link2ultrasonic_7']['roll']} ${calibration['base_link2ultrasonic_7']['pitch']} ${calibration['base_link2ultrasonic_7']['yaw']}" />
-  </joint>
-  <joint name="rs16_camera" type="fixed">
-    <parent link="rs16" />
-    <child link="camera" />
-    <origin xyz="${calibration['rs162camera']['x']} ${calibration['rs162camera']['y']} ${calibration['rs162camera']['z']}" rpy="${calibration['rs162camera']['roll']} ${calibration['rs162camera']['pitch']} ${calibration['rs162camera']['yaw']}" />
-  </joint>
+  <!-- sensor kit -->
+  <xacro:include filename="sensor_kit.xacro"/>
+  <xacro:sensor_kit_macro parent="base_link">
+    <origin
+      xyz="${calibration['base_link']['sensor_kit_base_link']['x']}
+           ${calibration['base_link']['sensor_kit_base_link']['y']}
+           ${calibration['base_link']['sensor_kit_base_link']['z']}"
+      rpy="${calibration['base_link']['sensor_kit_base_link']['roll']}
+           ${calibration['base_link']['sensor_kit_base_link']['pitch']}
+           ${calibration['base_link']['sensor_kit_base_link']['yaw']}"
+    />
+  </xacro:sensor_kit_macro>
+  <!-- ultrasonic -->
+  <xacro:ultrasonic_0 >
+    <origin
+      xyz="${calibration['base_link']['ultrasonic_0']['x']}
+           ${calibration['base_link']['ultrasonic_0']['y']}
+           ${calibration['base_link']['ultrasonic_0']['z']}"
+      rpy="${calibration['base_link']['ultrasonic_0']['roll']}
+           ${calibration['base_link']['ultrasonic_0']['pitch']}
+           ${calibration['base_link']['ultrasonic_0']['yaw']}"
+    />
+  </xacro:ultrasonic_0>
+  <xacro:ultrasonic_1 >
+    <origin
+      xyz="${calibration['base_link']['ultrasonic_1']['x']}
+           ${calibration['base_link']['ultrasonic_1']['y']}
+           ${calibration['base_link']['ultrasonic_1']['z']}"
+      rpy="${calibration['base_link']['ultrasonic_1']['roll']}
+           ${calibration['base_link']['ultrasonic_1']['pitch']}
+           ${calibration['base_link']['ultrasonic_1']['yaw']}"
+    />
+  </xacro:ultrasonic_1>
+  <xacro:ultrasonic_2 >
+    <origin
+      xyz="${calibration['base_link']['ultrasonic_2']['x']}
+           ${calibration['base_link']['ultrasonic_2']['y']}
+           ${calibration['base_link']['ultrasonic_2']['z']}"
+      rpy="${calibration['base_link']['ultrasonic_2']['roll']}
+           ${calibration['base_link']['ultrasonic_2']['pitch']}
+           ${calibration['base_link']['ultrasonic_2']['yaw']}"
+    />
+  </xacro:ultrasonic_2>
+  <xacro:ultrasonic_3 >
+    <origin
+      xyz="${calibration['base_link']['ultrasonic_3']['x']}
+           ${calibration['base_link']['ultrasonic_3']['y']}
+           ${calibration['base_link']['ultrasonic_3']['z']}"
+      rpy="${calibration['base_link']['ultrasonic_3']['roll']}
+           ${calibration['base_link']['ultrasonic_3']['pitch']}
+           ${calibration['base_link']['ultrasonic_3']['yaw']}"
+    />
+  </xacro:ultrasonic_3>
+  <xacro:ultrasonic_4 >
+    <origin
+      xyz="${calibration['base_link']['ultrasonic_4']['x']}
+           ${calibration['base_link']['ultrasonic_4']['y']}
+           ${calibration['base_link']['ultrasonic_4']['z']}"
+      rpy="${calibration['base_link']['ultrasonic_4']['roll']}
+           ${calibration['base_link']['ultrasonic_4']['pitch']}
+           ${calibration['base_link']['ultrasonic_4']['yaw']}"
+    />
+  </xacro:ultrasonic_4>
+  <xacro:ultrasonic_5 >
+    <origin
+      xyz="${calibration['base_link']['ultrasonic_5']['x']}
+           ${calibration['base_link']['ultrasonic_5']['y']}
+           ${calibration['base_link']['ultrasonic_5']['z']}"
+      rpy="${calibration['base_link']['ultrasonic_5']['roll']}
+           ${calibration['base_link']['ultrasonic_5']['pitch']}
+           ${calibration['base_link']['ultrasonic_5']['yaw']}"
+    />
+  </xacro:ultrasonic_5>
+  <xacro:ultrasonic_6 >
+    <origin
+      xyz="${calibration['base_link']['ultrasonic_6']['x']}
+           ${calibration['base_link']['ultrasonic_6']['y']}
+           ${calibration['base_link']['ultrasonic_6']['z']}"
+      rpy="${calibration['base_link']['ultrasonic_6']['roll']}
+           ${calibration['base_link']['ultrasonic_6']['pitch']}
+           ${calibration['base_link']['ultrasonic_6']['yaw']}"
+    />
+  </xacro:ultrasonic_6>
+  <xacro:ultrasonic_7 >
+    <origin
+      xyz="${calibration['base_link']['ultrasonic_7']['x']}
+           ${calibration['base_link']['ultrasonic_7']['y']}
+           ${calibration['base_link']['ultrasonic_7']['z']}"
+      rpy="${calibration['base_link']['ultrasonic_7']['roll']}
+           ${calibration['base_link']['ultrasonic_7']['pitch']}
+           ${calibration['base_link']['ultrasonic_7']['yaw']}"
+    />
+  </xacro:ultrasonic_7>
 </robot>

Commit message: 添加ouster ultra fixposition的启动launch

File: pixkit_sensor_kit_description/urdf/sensors.xacro (robot description, xacro)
@@ -16,4 +16,8 @@
   <link name="ultrasonic_6" />
   <link name="ultrasonic_7" />
+  <link name="ultrasonic_8" />
+  <link name="ultrasonic_9" />
+  <link name="ultrasonic_10" />
+  <link name="ultrasonic_11" />
   <link name="camera" />
   <xacro:arg name="config_dir" default="$(find pixkit_sensor_kit_description)"/>
@@ -85,4 +89,24 @@
     <origin xyz="${calibration['base_link2ultrasonic_7']['x']} ${calibration['base_link2ultrasonic_7']['y']} ${calibration['base_link2ultrasonic_7']['z']}" rpy="${calibration['base_link2ultrasonic_7']['roll']} ${calibration['base_link2ultrasonic_7']['pitch']} ${calibration['base_link2ultrasonic_7']['yaw']}" />
   </joint>
+   <joint name="baselink_ultrasonic_8" type="fixed">
+    <parent link="base_link" />
+    <child link="ultrasonic_8" />
+    <origin xyz="${calibration['base_link2ultrasonic_8']['x']} ${calibration['base_link2ultrasonic_8']['y']} ${calibration['base_link2ultrasonic_8']['z']}" rpy="${calibration['base_link2ultrasonic_8']['roll']} ${calibration['base_link2ultrasonic_8']['pitch']} ${calibration['base_link2ultrasonic_8']['yaw']}" />
+  </joint>
+  <joint name="baselink_ultrasonic_9" type="fixed">
+    <parent link="base_link" />
+    <child link="ultrasonic_9" />
+    <origin xyz="${calibration['base_link2ultrasonic_9']['x']} ${calibration['base_link2ultrasonic_9']['y']} ${calibration['base_link2ultrasonic_9']['z']}" rpy="${calibration['base_link2ultrasonic_9']['roll']} ${calibration['base_link2ultrasonic_9']['pitch']} ${calibration['base_link2ultrasonic_9']['yaw']}" />
+  </joint>
+  <joint name="baselink_ultrasonic_10" type="fixed">
+    <parent link="base_link" />
+    <child link="ultrasonic_10" />
+    <origin xyz="${calibration['base_link2ultrasonic_10']['x']} ${calibration['base_link2ultrasonic_10']['y']} ${calibration['base_link2ultrasonic_10']['z']}" rpy="${calibration['base_link2ultrasonic_10']['roll']} ${calibration['base_link2ultrasonic_10']['pitch']} ${calibration['base_link2ultrasonic_10']['yaw']}" />
+  </joint>
+  <joint name="baselink_ultrasonic_11" type="fixed">
+    <parent link="base_link" />
+    <child link="ultrasonic_11" />
+    <origin xyz="${calibration['base_link2ultrasonic_11']['x']} ${calibration['base_link2ultrasonic_11']['y']} ${calibration['base_link2ultrasonic_11']['z']}" rpy="${calibration['base_link2ultrasonic_11']['roll']} ${calibration['base_link2ultrasonic_11']['pitch']} ${calibration['base_link2ultrasonic_11']['yaw']}" />
+  </joint>
   <joint name="rs16_camera" type="fixed">
     <parent link="rs16" />
