Commit message: fix:autoware整体启动修复

File: pixkit_sensor_kit_description/urdf/sensor_kit.xacro (robot description, xacro)
@@ -139,5 +139,5 @@
   <link name="ultrasonic_7" />
   <xacro:macro name="ultrasonic_0" params="*ultrasonic_origin parent=sensor_kit_base_link" >
-    <joint name="ultrasonic" type="fixed">
+    <joint name="ultrasonic_0_joint" type="fixed">
       <xacro:insert_block name="ultrasonic_origin"/>
       <parent link="${parent}"/>
@@ -146,5 +146,5 @@
   </xacro:macro>
   <xacro:macro name="ultrasonic_1" params="*ultrasonic_origin parent=sensor_kit_base_link" >
-    <joint name="ultrasonic" type="fixed">
+    <joint name="ultrasonic_1_joint" type="fixed">
       <xacro:insert_block name="ultrasonic_origin"/>
       <parent link="${parent}"/>
@@ -153,5 +153,5 @@
   </xacro:macro>
   <xacro:macro name="ultrasonic_2" params="*ultrasonic_origin parent=sensor_kit_base_link" >
-    <joint name="ultrasonic" type="fixed">
+    <joint name="ultrasonic_2_joint" type="fixed">
       <xacro:insert_block name="ultrasonic_origin"/>
       <parent link="${parent}"/>
@@ -160,5 +160,5 @@
   </xacro:macro>
   <xacro:macro name="ultrasonic_3" params="*ultrasonic_origin parent=sensor_kit_base_link" >
-    <joint name="ultrasonic" type="fixed">
+    <joint name="ultrasonic_3_joint" type="fixed">
       <xacro:insert_block name="ultrasonic_origin"/>
       <parent link="${parent}"/>
@@ -167,5 +167,5 @@
   </xacro:macro>
   <xacro:macro name="ultrasonic_4" params="*ultrasonic_origin parent=sensor_kit_base_link" >
-    <joint name="ultrasonic" type="fixed">
+    <joint name="ultrasonic_4_joint" type="fixed">
       <xacro:insert_block name="ultrasonic_origin"/>
       <parent link="${parent}"/>
@@ -174,5 +174,5 @@
   </xacro:macro>
   <xacro:macro name="ultrasonic_5" params="*ultrasonic_origin parent=sensor_kit_base_link" >
-    <joint name="ultrasonic" type="fixed">
+    <joint name="ultrasonic_5_joint" type="fixed">
       <xacro:insert_block name="ultrasonic_origin"/>
       <parent link="${parent}"/>
@@ -181,5 +181,5 @@
   </xacro:macro>
   <xacro:macro name="ultrasonic_6" params="*ultrasonic_origin parent=sensor_kit_base_link" >
-    <joint name="ultrasonic" type="fixed">
+    <joint name="ultrasonic_6_joint" type="fixed">
       <xacro:insert_block name="ultrasonic_origin"/>
       <parent link="${parent}"/>
@@ -188,5 +188,5 @@
   </xacro:macro>
   <xacro:macro name="ultrasonic_7" params="*ultrasonic_origin parent=sensor_kit_base_link" >
-    <joint name="ultrasonic" type="fixed">
+    <joint name="ultrasonic_7_joint" type="fixed">
       <xacro:insert_block name="ultrasonic_origin"/>
       <parent link="${parent}"/>

Commit message: feat：实车测试

File: pixkit_sensor_kit_description/urdf/sensor_kit.xacro (robot description, xacro)
@@ -15,6 +15,5 @@
     <!-- sensor -->
     <xacro:property name="calibration" value="${xacro.load_yaml('$(arg config_dir)/sensor_kit_calibration.yaml')}"/>
-    <link name="traffic_light_left_camera" />
-    <link name="zed" />
+    <link name="camera_top_link" />
     <link name="gnss" />
     <link name="laser_top_base_link" />
@@ -70,25 +69,14 @@
     </joint>
     <!-- camera -->
-    <joint name="traffic_light_left_camera_joint" type="fixed">
-      <parent link="sensor_kit_base_link" />
-      <child link="traffic_light_left_camera" />
+    <joint name="camera_top_link_joint" type="fixed">
+      <parent link="ouster_top_base_link" />
+      <child link="camera_top_link" />
       <origin
-        xyz="${calibration['sensor_kit_base_link']['traffic_light_left_camera']['x']}
-             ${calibration['sensor_kit_base_link']['traffic_light_left_camera']['y']}
-             ${calibration['sensor_kit_base_link']['traffic_light_left_camera']['z']}"
-        rpy="${calibration['sensor_kit_base_link']['traffic_light_left_camera']['roll']}
-             ${calibration['sensor_kit_base_link']['traffic_light_left_camera']['pitch']}
-             ${calibration['sensor_kit_base_link']['traffic_light_left_camera']['yaw']}" />
-    </joint>
-    <joint name="zed_joint" type="fixed">
-      <parent link="sensor_kit_base_link" />
-      <child link="zed" />
-      <origin
-        xyz="${calibration['sensor_kit_base_link']['zed']['x']}
-             ${calibration['sensor_kit_base_link']['zed']['y']}
-             ${calibration['sensor_kit_base_link']['zed']['z']}"
-        rpy="${calibration['sensor_kit_base_link']['zed']['roll']}
-             ${calibration['sensor_kit_base_link']['zed']['pitch']}
-             ${calibration['sensor_kit_base_link']['zed']['yaw']}" />
+        xyz="${calibration['ouster_top_base_link']['camera_top_link']['x']}
+             ${calibration['ouster_top_base_link']['camera_top_link']['y']}
+             ${calibration['ouster_top_base_link']['camera_top_link']['z']}"
+        rpy="${calibration['ouster_top_base_link']['camera_top_link']['roll']}
+             ${calibration['ouster_top_base_link']['camera_top_link']['pitch']}
+             ${calibration['ouster_top_base_link']['camera_top_link']['yaw']}" />
     </joint>
     <!-- gnss -->
